File: E-CAD/Thermostat/Thermostat.sch (KiCad schematic (older format))
At the start: 30 parts, among them IC3 CPC1972GSTR, J1 Screw_Terminal_01x04, J2 Conn_01x04_Female_Display, J3 Conn_01x04_Female_Prog, J4 Conn_01x07_Male, J5 Conn_01x02_Male, J6 Conn_01x03_Male, J7 Conn_01x03_Male_DHT, Q1 BC847, Q2 BC847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

Commit message: adjusting to api v3 and home assistant
Parts:
- IC3: symbol CPC1972GSTR:CPC1972GSTR -> Thermostat-rescue:CPC1972GSTR-CPC1972GSTR
- J1: symbol conn:Screw_Terminal_01x05 -> Thermostat-rescue:Screw_Terminal_01x05-conn
- J2: symbol conn:Conn_01x04_Female -> Thermostat-rescue:Conn_01x04_Female-conn
- J3: symbol conn:Conn_01x06_Female -> Thermostat-rescue:Conn_01x06_Female-conn
- J4: symbol conn:Conn_01x07_Male -> Thermostat-rescue:Conn_01x07_Male-conn
- J5: symbol conn:Conn_01x02_Male -> Thermostat-rescue:Conn_01x02_Male-conn
- J6, J7: symbol conn:Conn_01x03_Male -> Thermostat-rescue:Conn_01x03_Male-conn
- S1, S2: symbol K6-1212A-03:K6-1212A-03 -> Thermostat-rescue:K6-1212A-03-K6-1212A-03
- S4, S5: symbol TS-1187A-B-A-B:TS-1187A-B-A-B -> Thermostat-rescue:TS-1187A-B-A-B-TS-1187A-B-A-B
- U2: symbol mypower:TENSTAR_3.3 -> Thermostat-rescue:TENSTAR_3.3-mypower
Changed lines of the file:
@@
 $EndComp
 $Comp
-L mypower:TENSTAR_3.3 U2
+L Thermostat-rescue:TENSTAR_3.3-mypower U2
 U 1 1 61F71185
 P 8500 2750
@@
 	-1   0    0    1
 $EndComp
-Text GLabel 1750 1050 3    50   Input ~ 0
-SDA
-Text GLabel 1650 1050 3    50   Input ~ 0
-SCL
-$Comp
-L power:GND #PWR0105
-U 1 1 61F79E4B
-P 1450 1050
-F 0 "#PWR0105" H 1450 800 50  0001 C CNN
-F 1 "GND" H 1455 877 50  0000 C CNN
-F 2 "" H 1450 1050 50  0001 C CNN
-F 3 "" H 1450 1050 50  0001 C CNN
-	1    1450 1050
-	1    0    0    -1
-$EndComp
-$Comp
-L power:+3.3V #PWR0106
-U 1 1 61F7AB02
-P 1550 1300
-F 0 "#PWR0106" H 1550 1150 50  0001 C CNN
-F 1 "+3.3V" H 1565 1473 50  0000 C CNN
-F 2 "" H 1550 1300 50  0001 C CNN
-F 3 "" H 1550 1300 50  0001 C CNN
-	1    1550 1300
-	-1   0    0    1
-$EndComp
-Wire Wire Line
-	1550 1300 1550 1050
 Wire Wire Line
 	4700 1550 4700 1000
@@
 SCL
 $Comp
-L conn:Screw_Terminal_01x05 J1
+L Thermostat-rescue:Screw_Terminal_01x05-conn J1
 U 1 1 61F7C7CA
 P 7650 1400
@@
 $EndComp
 $Comp
-L conn:Conn_01x06_Female J3
+L Thermostat-rescue:Conn_01x06_Female-conn J3
 U 1 1 6200F70B
 P 2250 2250
@@
 	3600 1750 4100 1750
 $Comp
-L TS-1187A-B-A-B:TS-1187A-B-A-B S4
+L Thermostat-rescue:TS-1187A-B-A-B-TS-1187A-B-A-B S4
 U 1 1 620FAFEC
 P 5000 6200
@@
 Connection ~ 5000 5800
 $Comp
-L TS-1187A-B-A-B:TS-1187A-B-A-B S5
+L Thermostat-rescue:TS-1187A-B-A-B-TS-1187A-B-A-B S5
 U 1 1 62102DD0
 P 6950 6200
@@
 	5000 5800 6950 5800
 $Comp
-L CPC1972GSTR:CPC1972GSTR IC3
+L Thermostat-rescue:CPC1972GSTR-CPC1972GSTR IC3
 U 1 1 621084DD
 P 7050 4200
@@
 NoConn ~ 8150 6300
 $Comp
-L K6-1212A-03:K6-1212A-03 S1
+L Thermostat-rescue:K6-1212A-03-K6-1212A-03 S1
 U 1 1 6211AD27
 P 2900 6500
@@
 Earth
 $Comp
-L conn:Conn_01x07_Male J4
+L Thermostat-rescue:Conn_01x07_Male-conn J4
 U 1 1 6214A367
 P 3350 4850
@@
 $EndComp
 $Comp
-L conn:Conn_01x03_Male J6
+L Thermostat-rescue:Conn_01x03_Male-conn J6
 U 1 1 6214CC8C
 P 4450 5050
@@
 $EndComp
 $Comp
-L conn:Conn_01x02_Male J5
+L Thermostat-rescue:Conn_01x02_Male-conn J5
 U 1 1 6214F2A0
 P 3600 3200
@@
 $EndComp
 $Comp
-L conn:Conn_01x03_Male J7
+L Thermostat-rescue:Conn_01x03_Male-conn J7
 U 1 1 62156544
 P 5850 5100
@@
 DHT
 $Comp
-L conn:Conn_01x04_Female J2
+L Thermostat-rescue:Conn_01x04_Female-conn J2
 U 1 1 61F73F4C
 P 1550 850
@@
 AC_L
 $Comp
-L K6-1212A-03:K6-1212A-03 S2
+L Thermostat-rescue:K6-1212A-03-K6-1212A-03 S2
 U 1 1 6210D216
 P 1450 6500
@@
 Wire Wire Line
 	3300 7400 4400 7400
+Wire Wire Line
+	1550 1300 1550 1050
+$Comp
+L power:+3.3V #PWR0106
+U 1 1 61F7AB02
+P 1550 1300
+F 0 "#PWR0106" H 1550 1150 50  0001 C CNN
+F 1 "+3.3V" H 1565 1473 50  0000 C CNN
+F 2 "" H 1550 1300 50  0001 C CNN
+F 3 "" H 1550 1300 50  0001 C CNN
+	1    1550 1300
+	-1   0    0    1
+$EndComp
+Text GLabel 1650 1050 3    50   Input ~ 0
+SCL
+Text GLabel 1750 1050 3    50   Input ~ 0
+SDA
+$Comp
+L power:GND #PWR0105
+U 1 1 61F79E4B
+P 1450 1050
+F 0 "#PWR0105" H 1450 800 50  0001 C CNN
+F 1 "GND" H 1455 877 50  0000 C CNN
+F 2 "" H 1450 1050 50  0001 C CNN
+F 3 "" H 1450 1050 50  0001 C CNN
+	1    1450 1050
+	1    0    0    -1
+$EndComp
 $EndSCHEMATC
